Commit message: Update turtlebot3_burger.urdf.xacro

File: robot/Camera_model/turtlebot3_burger.urdf.xacro (robot description, xacro)
@@ -164,5 +164,5 @@
  <joint name="camera_joint" type="fixed">
     <axis xyz="0 1 0" />
-    <origin xyz="-0.09 0 0.1" rpy="0 0.5233 3.14"/> <!--position et orientation de la camera-->
+    <origin xyz="-0.09 0 0.1" rpy="0 0.17453292 3.1415926"/> <!--position et orientation de la camera-->
     <parent link="base_link"/>
     <child link="camera_link"/>

Commit message: Update turtlebot3_burger.urdf.xacro

File: robot/Camera_model/turtlebot3_burger.urdf.xacro (robot description, xacro)
@@ -164,5 +164,5 @@
  <joint name="camera_joint" type="fixed">
     <axis xyz="0 1 0" />
-    <origin xyz="-0.09 0 0.1" rpy="0 0.17453292 3.1415926"/> <!--position et orientation de la camera-->
+    <origin xyz="0.03 0 0.1" rpy="0 -0.17453292 3.1415926"/> <!--position et orientation de la camera-->
     <parent link="base_link"/>
     <child link="camera_link"/>

Commit message: Update turtlebot3_burger.urdf.xacro

File: robot/Camera_model/turtlebot3_burger.urdf.xacro (robot description, xacro)
@@ -164,5 +164,5 @@
  <joint name="camera_joint" type="fixed">
     <axis xyz="0 1 0" />
-    <origin xyz="0.03 0 0.1" rpy="0 -0.17453292 3.1415926"/> <!--position et orientation de la camera-->
+    <origin xyz="0.03 0 0.1" rpy="0 -0.17453292 0"/> <!--position et orientation de la camera-->
     <parent link="base_link"/>
     <child link="camera_link"/>

Commit message: Update turtlebot3_burger.urdf.xacro

File: robot/Camera_model/turtlebot3_burger.urdf.xacro (robot description, xacro)
@@ -164,5 +164,5 @@
  <joint name="camera_joint" type="fixed">
     <axis xyz="0 1 0" />
-    <origin xyz="0.03 0 0.1" rpy="0 -0.17453292 0"/> <!--position et orientation de la camera-->
+    <origin xyz="0.03 0 0.1" rpy="0 0.17453292 0"/> <!--position et orientation de la camera-->
     <parent link="base_link"/>
     <child link="camera_link"/>

Commit message: Update turtlebot3_burger.urdf.xacro

File: robot/Camera_model/turtlebot3_burger.urdf.xacro (robot description, xacro)
@@ -164,5 +164,5 @@
  <joint name="camera_joint" type="fixed">
     <axis xyz="0 1 0" />
-    <origin xyz="0.03 0 0.1" rpy="0 0.17453292 0"/> <!--position et orientation de la camera-->
+    <origin xyz="0.03 0 0.125" rpy="0 0.17453292 0"/> <!--position et orientation de la camera-->
     <parent link="base_link"/>
     <child link="camera_link"/>

Commit message: Update turtlebot3_burger.urdf.xacro

File: robot/Camera_model/turtlebot3_burger.urdf.xacro (robot description, xacro)
@@ -164,5 +164,5 @@
  <joint name="camera_joint" type="fixed">
     <axis xyz="0 1 0" />
-    <origin xyz="0.03 0 0.125" rpy="0 0.17453292 0"/> <!--position et orientation de la camera-->
+    <origin xyz="0.03 0 0.125" rpy="0 0.610865238 0"/> <!--position et orientation de la camera-->
     <parent link="base_link"/>
     <child link="camera_link"/>
